File: control-board/control-board.kicad_sch (KiCad schematic)
At the start: 0 parts

Commit message: Added screen, pi pico (for now), and the power reg
Signed-off-by: Ravinder Olivier Singh Dadiala <ravinder-Olivier@outlook.com>
Parts:
- added A1: RaspberryPi_Pico, Module:RaspberryPi_Pico_Common_Unspecified, symbol MCU_Module:RaspberryPi_Pico
- added C1: 1uF, symbol Device:C_45deg
- added C2: 1uF, symbol Device:C
- added C3, C5, C6: 0.1uF, symbol Device:C
- added C4: 10uF, symbol Device:C_Polarized
- added D1: 1N4007, Diode_THT:D_DO-41_SOD81_P10.16mm_Horizontal, symbol Diode:1N4007
- added D2: 1N5239, symbol Device:D_Zener
- added RN1: 150R, symbol Device:R_Pack07
- added U2: LM7805_TO220, Package_TO_SOT_THT:TO-220-3_Vertical, symbol Regulator_Linear:LM7805_TO220
- added U3: LD1117V33, Package_TO_SOT_THT:TO-220-3_Vertical, symbol Regulator_Linear:LD1117V33
- added U4: 74HC595, symbol 74xx:74HC595
- added U5: D168K, Display_7Segment:D1X8K, symbol Display_Character:D168K
Connections:
- new net: C3.1, C4.1, C5.1, C6.1, U3.2 (VO)
- new net: C2.1, U2.3 (VO), U3.3 (VI)
- new net: RN1.1 (R1.1), U5.10 (G)
- new net: RN1.10 (R5.2), U4.2 (QC)
- new net: RN1.11 (R4.2), U4.3 (QD)
- new net: RN1.12 (R3.2), U4.4 (QE)
- new net: RN1.13 (R2.2), U4.5 (QF)
- new net: RN1.14 (R1.2), U4.6 (QG)
- new net: RN1.2 (R2.1), U5.9 (F)
- new net: RN1.3 (R3.1), U5.1 (E)
- new net: RN1.4 (R4.1), U5.2 (D)
- new net: RN1.5 (R5.1), U5.4 (C)
- new net: RN1.6 (R6.1), U5.6 (B)
- new net: RN1.7 (R7.1), U5.7 (A)
- new net: RN1.8 (R7.2), U4.15 (QA)
- new net: RN1.9 (R6.2), U4.1 (QB)
- new net: A1.21 (GPIO16), U4.14 (SER)
- new net: A1.22 (GPIO17), U4.11 (SRCLK)
- new net: A1.24 (GPIO18), U4.12 (RCLK)
- new net: A1.39 (VSYS), C6.2
- new net: C1.2, D1.1 (K), D2.1 (K), U2.1 (VI)
- new net: C5.2, U4.10 (~{SRCLR}), U4.16 (VCC)
- new net +9V: D1.2 (A)
- new net GND: A1.13 (GND), A1.18 (GND), A1.23 (GND), A1.28 (GND), A1.3 (GND), A1.33 (AGND), A1.38 (GND), A1.8 (GND), C1.1, C2.2, C3.2, C4.2, D2.2 (A), U2.2 (GND), U3.1 (GND), U4.13 (~{OE}), U4.8 (GND), U5.3 (CC), U5.8 (CC)
Other:
- note added: "4114R-1-151LF"
- note added: "POWER REGULATION 9V -> 3.3V VERSION 2: MAX 800MA"
- note added: "SCREEN MODULE VERSION 1"
